Commit message: working basics

File: hoverboard-driver-hestia/description/urdf/diffbot_description.urdf.xacro (robot description, xacro)
@@ -2,123 +2,4 @@
 <robot xmlns:xacro="http://www.ros.org/wiki/xacro">
   <xacro:macro name="diffbot" params="prefix">
-  <!-- Constants for robot dimensions -->
-  <xacro:property name="PI" value="3.1415926535897931"/>
-  <xacro:property name="base_mass" value="1.0" /> <!-- arbitrary value for base mass -->
-  <xacro:property name="base_width" value="0.6" />
-  <xacro:property name="base_length" value="0.52" />
-  <xacro:property name="base_height" value="0.72" />
-  <xacro:property name="wheel_mass" value="0.3" /> <!-- arbitrary value for wheel mass -->
-  <xacro:property name="wheel_len" value="0.053" />
-  <xacro:property name="wheel_radius" value="0.0825" />
-  <xacro:property name="caster_wheel_mass" value="0.1" /> <!-- arbitrary value for caster wheel mass -->
-  <xacro:property name="caster_wheel_radius" value="0.04" />
-  <xacro:property name="z_offset" value="0" /> <!-- Space btw top of beam and the each joint -->
-  <!-- Base Link -->
-  <link name="${prefix}base_link">
-    <collision>
-      <origin xyz="0 0 ${base_height/2}" rpy="0 0 0"/>
-      <geometry>
-        <box size="${base_width} ${base_length} ${base_height}"/>
-      </geometry>
-    </collision>
-    <visual>
-      <origin xyz="0 0 ${base_height/2}" rpy="0 0 0"/>
-      <geometry>
-        <box size="${base_width} ${base_length} ${base_height}"/>
-      </geometry>
-      <material name="orange"/>
-    </visual>
-    <inertial>
-      <origin xyz="0 0 0" rpy="0 0 0"/>
-      <mass value="${base_mass}"/>
-      <inertia
-        ixx="${base_mass / 12.0 * (base_length*base_length + base_height*base_height)}" ixy="0.0" ixz="0.0"
-        iyy="${base_mass / 12.0 * (base_height*base_height + base_width*base_width)}" iyz="0.0"
-        izz="${base_mass / 12.0 * (base_width*base_width + base_length*base_length)}"/>
-      </inertial>
-    </link>
-    <gazebo reference="${prefix}base_link">
-      <material>Gazebo/Orange</material>
-    </gazebo>
-    <joint name="${prefix}left_wheel_joint" type="continuous">
-      <parent link="${prefix}base_link"/>
-      <child link="${prefix}left_wheel"/>
-      <origin xyz="0 -0.15 ${z_offset}" rpy="0 0 0"/>
-      <axis xyz="0 1 0"/>
-      <dynamics damping="0.2"/>
-    </joint>
-    <!-- left wheel Link -->
-    <link name="${prefix}left_wheel">
-      <collision>
-        <origin xyz="0 0 0" rpy="${PI/2} 0 0"/>
-        <geometry>
-          <cylinder length="${wheel_len}" radius="${wheel_radius}"/>
-        </geometry>
-      </collision>
-      <visual>
-        <origin xyz="0 0 0" rpy="${PI/2} 0 0"/>
-        <geometry>
-          <cylinder length="${wheel_len}" radius="${wheel_radius}"/>
-        </geometry>
-        <material name="black"/>
-      </visual>
-      <inertial>
-        <origin xyz="0 0 0" rpy="${PI/2} 0 0"/>
-        <mass value="${wheel_mass}"/>
-        <inertia
-          ixx="${wheel_mass / 12.0 * (3*wheel_radius*wheel_radius + wheel_len*wheel_len)}" ixy="0.0" ixz="0.0"
-          iyy="${wheel_mass / 12.0 * (3*wheel_radius*wheel_radius + wheel_len*wheel_len)}" iyz="0.0"
-          izz="${wheel_mass / 2.0 * wheel_radius*wheel_radius}"/>
-        </inertial>
-      </link>
-      <gazebo reference="${prefix}left_wheel">
-          <material>Gazebo/Black</material>
-      </gazebo>
-    <joint name="${prefix}right_wheel_joint" type="continuous">
-      <parent link="${prefix}base_link"/>
-      <child link="${prefix}right_wheel"/>
-      <origin xyz="0 0.15 ${z_offset}" rpy="0 0 0"/>
-      <axis xyz="0 1 0"/>
-      <dynamics damping="0.2"/>
-    </joint>
-    <!-- right wheel Link -->
-    <link name="${prefix}right_wheel">
-      <collision>
-        <origin xyz="0 0 0" rpy="${PI/2} 0 0"/>
-        <geometry>
-          <cylinder length="${wheel_len}" radius="${wheel_radius}"/>
-        </geometry>
-      </collision>
-      <visual>
-        <origin xyz="0 0 0" rpy="${PI/2} 0 0"/>
-        <geometry>
-          <cylinder length="${wheel_len}" radius="${wheel_radius}"/>
-        </geometry>
-        <material name="black"/>
-      </visual>
-      <inertial>
-        <origin xyz="0 0 0" rpy="${PI/2} 0 0"/>
-        <mass value="${wheel_mass}"/>
-        <inertia
-          ixx="${wheel_mass / 12.0 * (3*wheel_radius*wheel_radius + wheel_len*wheel_len)}" ixy="0.0" ixz="0.0"
-          iyy="${wheel_mass / 12.0 * (3*wheel_radius*wheel_radius + wheel_len*wheel_len)}" iyz="0.0"
-          izz="${wheel_mass / 2.0 * wheel_radius*wheel_radius}"/>
-        </inertial>
-      </link>
-      <gazebo reference="${prefix}right_wheel">
-          <material>Gazebo/Black</material>
-      </gazebo>
-  <!-- Include Caster Wheels -->
-  <xacro:include filename="$(find hoverboard_driver)/urdf/caster_wheels.urdf.xacro"/>
-  <!-- BASE_FOOTPRINT LINK -->
-  <joint name="base_footprint_joint" type="fixed">
-    <parent link="base_footprint"/>
-    <child link="${prefix}base_link"/>
-    <origin xyz="0 0 0" rpy="0 0 0"/>
-  </joint>
-  <link name="base_footprint">
-  </link>
-  <!-- Include Lidar -->
-  <xacro:include filename="$(find hoverboard_driver)/urdf/lidar.xacro" />
   </xacro:macro>
 </robot>

Commit message: Tf from xacro file

File: hoverboard-driver-hestia/description/urdf/diffbot_description.urdf.xacro (robot description, xacro)
@@ -1,5 +1,28 @@
 <?xml version="1.0"?>
-<robot xmlns:xacro="http://www.ros.org/wiki/xacro">
+<robot xmlns:xacro="http://www.ros.org/wiki/xacro" name="diffbot_robot">
   <xacro:macro name="diffbot" params="prefix">
+    <!-- base_footprint -->
+    <link name="${prefix}base_footprint"/>
+    <!-- base_link -->
+    <link name="${prefix}base_link"/>
+    <joint name="${prefix}base_footprint_to_base_link" type="fixed">
+      <parent link="${prefix}base_footprint"/>
+      <child link="${prefix}base_link"/>
+      <origin xyz="0 -0.08 0" rpy="0 0 0"/>
+    </joint>
+    <!-- laser -->
+    <link name="${prefix}laser"/>
+    <joint name="${prefix}base_link_to_laser" type="fixed">
+      <parent link="${prefix}base_link"/>
+      <child link="${prefix}laser"/>
+      <origin xyz="-0.35 0 0.06" rpy="0 0 0"/>
+    </joint>
+    <!-- scan (often optional) -->
+    <link name="${prefix}scan"/>
+    <joint name="${prefix}laser_to_scan" type="fixed">
+      <parent link="${prefix}laser"/>
+      <child link="${prefix}scan"/>
+      <origin xyz="0 0 0" rpy="0 0 0"/>
+    </joint>
   </xacro:macro>
 </robot>

Commit message: adjusted tf

File: hoverboard-driver-hestia/description/urdf/diffbot_description.urdf.xacro (robot description, xacro)
@@ -9,5 +9,5 @@
       <parent link="${prefix}base_footprint"/>
       <child link="${prefix}base_link"/>
-      <origin xyz="0 -0.08 0" rpy="0 0 0"/>
+      <origin xyz="0.20 0 0" rpy="0 0 0"/>
     </joint>
     <!-- laser -->
@@ -16,5 +16,5 @@
       <parent link="${prefix}base_link"/>
       <child link="${prefix}laser"/>
-      <origin xyz="-0.35 0 0.06" rpy="0 0 0"/>
+      <origin xyz="0.2 0 0.06" rpy="0 0 0"/>
     </joint>
     <!-- scan (often optional) -->

Commit message: Saving

File: hoverboard-driver-hestia/description/urdf/diffbot_description.urdf.xacro (robot description, xacro)
@@ -9,5 +9,5 @@
       <parent link="${prefix}base_footprint"/>
       <child link="${prefix}base_link"/>
-      <origin xyz="0.20 0 0" rpy="0 0 0"/>
+      <origin xyz="0 0 0" rpy="0 0 0"/>
     </joint>
     <!-- laser -->

Commit message: first tests

File: hoverboard-driver-hestia/description/urdf/diffbot_description.urdf.xacro (robot description, xacro)
@@ -11,11 +11,11 @@
       <origin xyz="0 0 0" rpy="0 0 0"/>
     </joint>
-    <!-- laser -->
-    <link name="${prefix}laser"/>
-    <joint name="${prefix}base_link_to_laser" type="fixed">
-      <parent link="${prefix}base_link"/>
-      <child link="${prefix}laser"/>
-      <origin xyz="0.2 0 0.06" rpy="0 0 0"/>
-    </joint>
+<!-- laser -->
+<link name="${prefix}laser"/>
+<joint name="${prefix}base_link_to_laser" type="fixed">
+  <parent link="${prefix}base_link"/>
+  <child link="${prefix}laser"/>
+  <origin xyz="0.2 0 0.06" rpy="0 0 3.14159"/>
+</joint>
     <!-- scan (often optional) -->
     <link name="${prefix}scan"/>

Commit message: box filter ajustado mas nao funcionando

File: hoverboard-driver-hestia/description/urdf/diffbot_description.urdf.xacro (robot description, xacro)
@@ -11,11 +11,11 @@
       <origin xyz="0 0 0" rpy="0 0 0"/>
     </joint>
-<!-- laser -->
-<link name="${prefix}laser"/>
-<joint name="${prefix}base_link_to_laser" type="fixed">
-  <parent link="${prefix}base_link"/>
-  <child link="${prefix}laser"/>
-  <origin xyz="0.2 0 0.06" rpy="0 0 3.14159"/>
-</joint>
+    <!-- laser -->
+    <link name="${prefix}laser"/>
+    <joint name="${prefix}base_link_to_laser" type="fixed">
+      <parent link="${prefix}base_link"/>
+      <child link="${prefix}laser"/>
+      <origin xyz="0.2 0 0.06" rpy="0 0 3.14159"/>
+    </joint>
     <!-- scan (often optional) -->
     <link name="${prefix}scan"/>
@@ -25,4 +25,11 @@
       <origin xyz="0 0 0" rpy="0 0 0"/>
     </joint>
+    <!-- base_scan -->
+    <!-- <link name="${prefix}base_scan"/>
+    <joint name="${prefix}laser_to_scan" type="fixed">
+      <parent link="${prefix}laser"/>
+      <child link="${prefix}base_scan"/>
+      <origin xyz="0 0 0" rpy="0 0 0"/>
+    </joint> -->
   </xacro:macro>
 </robot>

Commit message: sucessful basic map and nav configs

File: hoverboard-driver-hestia/description/urdf/diffbot_description.urdf.xacro (robot description, xacro)
@@ -16,5 +16,5 @@
       <parent link="${prefix}base_link"/>
       <child link="${prefix}laser"/>
-      <origin xyz="0.2 0 0.06" rpy="0 0 3.14159"/>
+      <origin xyz="0.15 0 0.06" rpy="0 0 3.14159"/>
     </joint>
     <!-- scan (often optional) -->
@@ -25,11 +25,4 @@
       <origin xyz="0 0 0" rpy="0 0 0"/>
     </joint>
-    <!-- base_scan -->
-    <!-- <link name="${prefix}base_scan"/>
-    <joint name="${prefix}laser_to_scan" type="fixed">
-      <parent link="${prefix}laser"/>
-      <child link="${prefix}base_scan"/>
-      <origin xyz="0 0 0" rpy="0 0 0"/>
-    </joint> -->
   </xacro:macro>
 </robot>

Commit message: cbr params

File: hoverboard-driver-hestia/description/urdf/diffbot_description.urdf.xacro (robot description, xacro)
@@ -16,5 +16,5 @@
       <parent link="${prefix}base_link"/>
       <child link="${prefix}laser"/>
-      <origin xyz="0.15 0 0.06" rpy="0 0 3.14159"/>
+      <origin xyz="0.18 0 0.06" rpy="0 0 3.14159"/>
     </joint>
     <!-- scan (often optional) -->
